Commit message: updated documentation with task done

File: src/my_robot_description/urdf/rubot/rubot_custom.urdf (robot description, URDF)
Before this commit: robot rubot, 9 links, 8 joints
Links:
- added link number2_link, mass 0.005; collision box size=0.03 0.03 0.02; visual mesh filename=file://$(find my_robot_description)/meshes/rubot/number_2.s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 scale=0.0006 0.0006 0.0006
Joints:
- added joint joint_number2: type fixed, parent base_link, child number2_link, origin xyz=0.08 0.0 0.14 rpy=0 0 0

Commit message: trial object3D in rubot_custom.urdf

File: src/my_robot_description/urdf/rubot/rubot_custom.urdf (robot description, URDF)
Before this commit: robot rubot, 10 links, 9 joints
Links:
- added link object3D_link, mass 0.02; collision box size=0.05 0.05 0.05; visual mesh filename=file://$(find my_robot_description)/meshes/rubot/object3D.s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 scale=0.05 0.05 0.05
Joints:
- added joint joint_object3D: type fixed, parent base_link, child object3D_link, origin xyz=0.0 0.0 0.1 rpy=0 0 0

Commit message: goodboy v2 ;)

File: src/my_robot_description/urdf/rubot/rubot_custom.urdf (robot description, URDF)
Before this commit: robot rubot, 11 links, 10 joints
Links:
- link object3D_link: mass 0.02 -> 0.01; geometry collision mesh filename=file://$(find my_robot_description)/meshes/rubot/object3D.s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 scale=0.000012 0.000012 0.000012; visual mesh filename=file://$(find my_robot_description)/meshes/rubot/object3D.s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 scale=0.000012 0.000012 0.000012
Joints:
- joint joint_object3D: origin xyz=0.0 0.0 0.1 rpy=0 0 0 -> xyz=0.015 0.0 0.1445 rpy=0 0 90
