Commit message: start doing MD and changes in URDF

File: src/my_robot_description/urdf/rubot/rubot_mecanum_lidar.urdf (robot description, URDF)
Before this commit: robot rubot, 11 links, 10 joints
Links:
- removed link number2_link
- removed link object3D_link
Joints:
- removed joint joint_number2
- removed joint joint_object3D
